File: PS2Keyboard.kicad_sch (KiCad schematic)
At the start: 13 parts, among them J1 KEYBOARD, U10 74HC32, U11 74HC14, U12 74HC00, U13 74595, U14 74595

Commit message: Misc Updates/Cleanup
Parts:
- C1, C28: value 0.01µF -> 0.1µF; footprint Capacitor_THT:C_Disc_D3.8mm_W2.6mm_P2.50mm -> Capacitor_THT:C_Disc_D5.0mm_W2.5mm_P2.50mm
- R12: value 1k -> 100
- R4: value 3k3 -> 330
- U10: value 74HC32 -> 74HCT32
- U11: value 74HC14 -> 74HCT14
- U12: value 74HC00 -> 74HCT00
- U13, U14: value 74595 -> 74HCT595
Changed lines of the file:
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@@
       (effects (font (size 1.27 1.27)))
     )
-    (property "Value" "74595" (at 225.425 106.045 0)
+    (property "Value" "74HCT595" (at 225.425 106.045 0)
       (effects (font (size 1.27 1.27)) (justify right))
     )
@@
       (effects (font (size 1.27 1.27)))
     )
-    (property "Value" "74595" (at 191.135 106.045 0)
+    (property "Value" "74HCT595" (at 191.135 106.045 0)
       (effects (font (size 1.27 1.27)) (justify right))
     )
@@
       (effects (font (size 1.27 1.27)))
     )
-    (property "Value" "74HC14" (at 128.905 73.025 0)
+    (property "Value" "74HCT14" (at 128.905 73.025 0)
       (effects (font (size 1.27 1.27)))
     )
@@
       (effects (font (size 1.27 1.27)))
     )
-    (property "Value" "74HC14" (at 128.905 88.265 0)
+    (property "Value" "74HCT14" (at 128.905 88.265 0)
       (effects (font (size 1.27 1.27)))
     )
@@
       (effects (font (size 1.27 1.27)))
     )
-    (property "Value" "74HC14" (at 78.105 93.345 0)
+    (property "Value" "74HCT14" (at 78.105 93.345 0)
       (effects (font (size 1.27 1.27)))
     )
@@
       (effects (font (size 1.27 1.27)) (justify left))
     )
-    (property "Value" "3k3" (at 140.7922 75.438 0)
+    (property "Value" "330" (at 140.7922 75.438 0)
       (effects (font (size 1.27 1.27)) (justify left))
     )
@@
       (effects (font (size 1.27 1.27)) (justify left))
     )
-    (property "Value" "0.01µF" (at 152.146 90.678 0)
-      (effects (font (size 1.27 1.27)) (justify left))
-    )
-    (property "Footprint" "Capacitor_THT:C_Disc_D3.8mm_W2.6mm_P2.50mm" (at 150.1902 93.345 0)
+    (property "Value" "0.1µF" (at 152.146 90.678 0)
+      (effects (font (size 1.27 1.27)) (justify left))
+    )
+    (property "Footprint" "Capacitor_THT:C_Disc_D5.0mm_W2.5mm_P2.50mm" (at 150.1902 93.345 0)
       (effects (font (size 1.27 1.27)) hide)
     )
@@
       (effects (font (size 1.27 1.27)))
     )
-    (property "Value" "74HC32" (at 150.495 107.7214 0)
+    (property "Value" "74HCT32" (at 150.495 107.7214 0)
       (effects (font (size 1.27 1.27)))
     )
@@
       (effects (font (size 1.27 1.27)))
     )
-    (property "Value" "74HC14" (at 130.175 52.705 0)
+    (property "Value" "74HCT14" (at 130.175 52.705 0)
       (effects (font (size 1.27 1.27)))
     )
@@
       (effects (font (size 1.27 1.27)) (justify left))
     )
-    (property "Value" "1k" (at 105.283 89.9922 0)
+    (property "Value" "100" (at 105.283 89.9922 0)
       (effects (font (size 1.27 1.27)) (justify left))
     )
@@
       (effects (font (size 1.27 1.27)))
     )
-    (property "Value" "74HC14" (at 80.01 152.4 0)
+    (property "Value" "74HCT14" (at 80.01 152.4 0)
       (effects (font (size 1.27 1.27)))
     )
@@
       (effects (font (size 1.27 1.27)))
     )
-    (property "Value" "74HC00" (at 100.33 119.7864 0)
+    (property "Value" "74HCT00" (at 100.33 119.7864 0)
       (effects (font (size 1.27 1.27)))
     )
@@
       (effects (font (size 1.27 1.27)))
     )
-    (property "Value" "74HC00" (at 59.055 154.94 0)
+    (property "Value" "74HCT00" (at 59.055 154.94 0)
       (effects (font (size 1.27 1.27)))
     )
@@
       (effects (font (size 1.27 1.27)))
     )
-    (property "Value" "74HC00" (at 60.96 79.7814 0)
+    (property "Value" "74HCT00" (at 60.96 79.7814 0)
       (effects (font (size 1.27 1.27)))
     )
@@
       (effects (font (size 1.27 1.27)))
     )
-    (property "Value" "74HC00" (at 100.33 152.4 0)
+    (property "Value" "74HCT00" (at 100.33 152.4 0)
       (effects (font (size 1.27 1.27)))
     )
@@
       (effects (font (size 1.27 1.27)) (justify left))
     )
-    (property "Value" "0.01µF" (at 96.901 99.568 0)
-      (effects (font (size 1.27 1.27)) (justify left))
-    )
-    (property "Footprint" "Capacitor_THT:C_Disc_D3.8mm_W2.6mm_P2.50mm" (at 94.9452 102.235 0)
+    (property "Value" "0.1µF" (at 96.901 99.568 0)
+      (effects (font (size 1.27 1.27)) (justify left))
+    )
+    (property "Footprint" "Capacitor_THT:C_Disc_D5.0mm_W2.5mm_P2.50mm" (at 94.9452 102.235 0)
       (effects (font (size 1.27 1.27)) hide)
     )
@@
       (effects (font (size 1.27 1.27)))
     )
-    (property "Value" "74HC32" (at 43.815 133.7564 0)
-      (effects (font (size 1.27 1.27)))
-    )
+    (property "Value" "74HCT32" (at 43.815 133.7564 0)
+      (effects (font (size 1.27 1.27)))
+    )
