File: IRQDecoder.kicad_sch (KiCad schematic)
At the start: 6 parts, among them U17 74HC138, U18 74HC148, U20 74HC373, U4 74HC32

Commit message: Schematic cleanup
Other:
- moved on the sheet: RN2, U18, U20, U4C

Commit message: Misc Updates/Cleanup
Parts:
- U17: value 74HC138 -> 74HCT138
- U18: value 74HC148 -> 74HCT148
- U20: value 74HC373 -> 74HCT373
- U4: value 74HC32 -> 74HCT32
Changed lines of the file:
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@@
       (effects (font (size 1.27 1.27)))
     )
-    (property "Value" "74HC138" (at 72.39 173.355 0)
+    (property "Value" "74HCT138" (at 72.39 173.355 0)
       (effects (font (size 1.27 1.27)))
     )
@@
       (effects (font (size 1.27 1.27)))
     )
-    (property "Value" "74HC148" (at 133.985 61.595 0)
+    (property "Value" "74HCT148" (at 133.985 61.595 0)
       (effects (font (size 1.27 1.27)))
     )
@@
       (effects (font (size 1.27 1.27)))
     )
-    (property "Value" "74HC373" (at 182.245 59.055 0)
+    (property "Value" "74HCT373" (at 182.245 59.055 0)
       (effects (font (size 1.27 1.27)))
     )
@@
       (effects (font (size 1.27 1.27)) (justify right))
     )
-    (property "Value" "74HC32" (at 144.145 117.475 90)
+    (property "Value" "74HCT32" (at 144.145 117.475 90)
       (effects (font (size 1.27 1.27)) (justify right))
     )

Commit message: Work-in-progress
Parts:
- removed RN1: 10k, Resistor_THT:R_Array_SIP10, symbol Device:R_Network09_US
- removed U17: 74HCT138, Package_DIP:DIP-16_W7.62mm_LongPads, symbol 74xx:74LS138
- added C5: 0.1µF, Capacitor_THT:C_Disc_D5.0mm_W2.5mm_P2.50mm, symbol Device:C
- added U10: 74HCT688, Package_DIP:DIP-20_W7.62mm, symbol 74xx:74HCT688
- added U11: 74HCT139, Package_DIP:DIP-16_W7.62mm, symbol 74xx:74LS139
- U18: footprint Package_DIP:DIP-16_W7.62mm_LongPads -> Package_DIP:DIP-16_W7.62mm
- U20: footprint Package_DIP:DIP-20_W7.62mm_LongPads -> Package_DIP:DIP-20_W7.62mm
- U4: footprint Package_DIP:DIP-14_W7.62mm_LongPads -> Package_DIP:DIP-14_W7.62mm
Connections:
- net +5V: now also C5.1, U10.20 (VCC), U11.16 (VCC)
- net A5: now also U10.13 (P5)
- net A6: now also U10.15 (P6)
- net A7: now also U10.17 (P7)
- net GND: now also C5.2, U10.10 (GND), U10.12 (R4), U10.14 (R5), U10.16 (R6), U10.18 (R7), U10.2 (P0), U10.3 (R0), U10.4 (P1), U10.5 (R1), U10.6 (P2), U10.7 (R2), U10.9 (R3), U11.13 (A1), U11.14 (A0), U11.15 (E), U11.8 (GND)
- net ~{IORQ}: now also U10.1 (G)
- net ~{SLOT0}: now also U11.4 (O0)
- new net A1: U11.3 (A1)
- new net A2: U11.2 (A0)
- new net A3: U10.8 (P3)
- new net A4: U10.11 (P4)
- new net ~{INTERNAL_IO}: U10.19 (P=R), U11.1 (E)
- new net ~{KEYB}: U11.6 (O2)
- new net ~{NVRAM}: U11.5 (O1)
- new net ~{SERIAL}: U11.7 (O3)
- no-connect marks 2 -> 1
