File: Interis 64.kicad_pcb (KiCad board)
At the start: 2 copper layers, 228.6 x 127 mm, 94 parts, among them J1 KEYBOARD, J2 Ext. RESET, J4 DB9_Male, J7 POWER, SW1 RESET, U1 DS1233, U10 74HCT32, U11 74HCT14, U12 74HCT00, U13 74HCT595, U14 74HCT595, U15 MC6850, U16 MAX232, U17 74HCT138, U18 74HCT148, U19 74HCT92, U2 Z80B CPU, U20 74HCT373, U21 74HCT02, U22 DS12885+, U3 28C256, U4 74HCT32, U5 62256, U6 74HCT32, U7 74HCT00, U8 62256, U9 74HCT04, Y1 7.3728MHz, Y2 32.768kHz

Commit message: Work-in-progress
Parts:
- removed C12, C13, C28, C31: 0.1µF, Capacitor_THT:C_Disc_D5.0mm_W2.5mm_P2.50mm
- removed C24, C25, C26, C27: 10µF, Capacitor_THT:CP_Radial_D5.0mm_P2.00mm
- removed D1: 1N4001, Diode_THT:D_DO-41_SOD81_P10.16mm_Horizontal
- removed J1: KEYBOARD, Connector_JST:JST_XH_B6B-XH-A_1x06_P2.50mm_Vertical
- removed J7: POWER, Connector_TE-Connectivity:TE_MATE-N-LOK_350211-1_1x04_P5.08mm_Vertical
- removed R12: 100, Resistor_THT:R_Axial_DIN0207_L6.3mm_D2.5mm_P10.16mm_Horizontal
- removed R3, R5: 10k, Resistor_THT:R_Axial_DIN0207_L6.3mm_D2.5mm_P10.16mm_Horizontal
- removed R4: 330, Resistor_THT:R_Axial_DIN0207_L6.3mm_D2.5mm_P10.16mm_Horizontal
- removed RN1: 10k, Resistor_THT:R_Array_SIP10
- removed SLOT6: $C0-DF, Connector_PCBEdge:EDAC_345-030-520-201
- removed SLOT7: $E0-$FF, Connector_PCBEdge:EDAC_345-030-520-201
- removed SW1: RESET, Button_Switch_THT:SW_TH_Tactile_Omron_B3F-10xx
- removed TP3, TP5, TP8: GND, TestPoint:TestPoint_Loop_D2.60mm_Drill1.6mm_Beaded
- removed U13, U14: 74HCT595, Package_DIP:DIP-16_W7.62mm_LongPads
- removed U17: 74HCT138, Package_DIP:DIP-16_W7.62mm_LongPads
- removed U21: 74HCT02, Package_DIP:DIP-14_W7.62mm_LongPads
- added J3: Conn_01x04, Interis-Footprints:TE_EconomyPower_1744037-x_1x04_P5.08mm_Vertical, F.Cu at (38.1, 48.3)
- added J5: Conn_01x06, Connector_JST:JST_XH_B6B-XH-A_1x06_P2.50mm_Vertical, F.Cu at (75.7, 29.8)
- added REF**: OSHW-Logo_7.5x8mm_SilkScreen, Symbol:OSHW-Logo_7.5x8mm_SilkScreen, F.Cu at (216.5, 144.8)
- added SLOT2: $80-$9F, Connector_PCBEdge:Interis_DMA_Socket, F.Cu at (178.4, 62.2)
- added SLOT3: $80-$9F, Connector_PCBEdge:Interis_DMA_Socket, F.Cu at (198.8, 62.2)
- added SLOT4: $80-$9F, Connector_PCBEdge:Interis_DMA_Socket, F.Cu at (219.1, 62.2)
- added U23: VT82C42, Package_DIP:DIP-40_W15.24mm, F.Cu at (47.6, 33.0)
- added U24: 74HCT06, Package_DIP:DIP-14_W7.62mm, F.Cu at (70.5, 66.0)
- J2: value Ext. RESET -> ExtReset; footprint Connector_JST:JST_XH_B2B-XH-A_1x02_P2.50mm_Vertical -> Connector_JST:JST_XH_B4B-XH-A_1x04_P2.50mm_Vertical
- SLOT5: value $A0-BF -> $80-$9F; footprint Connector_PCBEdge:EDAC_345-030-520-201 -> Connector_PCBEdge:Interis_DMA_Socket
- U1: footprint Package_TO_SOT_THT:TO-92_Inline -> Package_TO_SOT_THT:TO-92_HandSolder
- U10: value 74HCT32 -> 74HCT688; footprint Package_DIP:DIP-14_W7.62mm_LongPads -> Package_DIP:DIP-20_W7.62mm
- U11: value 74HCT14 -> 74HCT139; footprint Package_DIP:DIP-14_W7.62mm_LongPads -> Package_DIP:DIP-16_W7.62mm
- U12: value 74HCT00 -> 74HCT32; footprint Package_DIP:DIP-14_W7.62mm_LongPads -> Package_DIP:DIP-14_W7.62mm
- U15, U22: footprint Package_DIP:DIP-24_W15.24mm_LongPads -> Package_DIP:DIP-24_W15.24mm
- U16, U18: footprint Package_DIP:DIP-16_W7.62mm_LongPads -> Package_DIP:DIP-16_W7.62mm
- U19, U4, U6, U7, U9: footprint Package_DIP:DIP-14_W7.62mm_LongPads -> Package_DIP:DIP-14_W7.62mm
- U2: footprint Package_DIP:DIP-40_W15.24mm_LongPads -> Package_DIP:DIP-40_W15.24mm
- U20: footprint Package_DIP:DIP-20_W7.62mm_LongPads -> Package_DIP:DIP-20_W7.62mm
- U3, U5, U8: footprint Package_DIP:DIP-28_W15.24mm_LongPads -> Package_DIP:DIP-28_W15.24mm
- moved C17 91.2 mm to (106.0, 54.6), turned to 180 degrees
- moved LS1 74.4 mm to (250.8, 133.9)
- moved JP3 66.5 mm to (252.1, 98.4), turned to 180 degrees
- moved JP1 64.1 mm to (113.0, 138.4), turned to 180 degrees
- moved Y2 57.0 mm to (244.5, 126.4)
- moved SLOT5 48.7 mm to (239.4, 62.2)
- moved C30 45.8 mm to (224.2, 102.2), turned to 0 degrees
- moved C18 44.3 mm to (190.5, 123.2)
- moved C1 41.8 mm to (90.8, 59.7), turned to 180 degrees
- moved U22 40.4 mm to (224.2, 120.6)
- moved U10 38.2 mm to (101.0, 58.4)
- moved U19 36.4 mm to (85.7, 40.6), turned to 0 degrees
- moved U18 34.2 mm to (196.2, 116.8)
- moved JP2 33.6 mm to (104.8, 30.5), turned to -90 degrees
- moved C32 31.1 mm to (111.1, 42.5), turned to -90 degrees
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- renumbered SLOT4 to SLOT1
Connections:
- C1 pad 1: Net-(D1-K) -> +5V
- J2 pad 1: ~{RESET} -> +5V
- JP1 pad 1: +5V -> Net-(JP1-A)
- JP1 pad 2: Net-(JP1-C) -> /Memory/~{A15}
- JP1 pad 3: ~{RAMLO} -> +5V
- SLOT1 pad a17: ~{NMI} -> ~{WAIT}
- SLOT1 pad a18: ~{BUSACK} -> ~{NMI}
- SLOT1 pad a19: ~{BUSRQ} -> ~{MREQ}
- SLOT1 pad a20: A6 -> ~{BUSRQ}
- SLOT1 pad a25: unconnected-(SLOT4-Pin_a25-Pada25) -> ~{RD}
- SLOT1 pad a5: unconnected-(SLOT4-Pin_a5-Pada5) -> A6
- SLOT1 pad a6: ~{RD} -> ~{WR}
- SLOT1 pad a7: ~{WR} -> ~{IRQ3}
- SLOT1 pad a8: ~{WAIT} -> ~{IRQ5}
- SLOT1 pad a9: CLOCK -> ~{IRQ7}
- SLOT1 pad b1: GND -> +12V
- SLOT1 pad b15: +5V -> GND
- SLOT1 pad b16: ~{RFSH} -> unconnected-(SLOT1-Pin_b16-Padb16)
- SLOT1 pad b17: ~{INT} -> ~{RESET}
- SLOT1 pad b18: ~{MREQ} -> ~{RFSH}
- SLOT1 pad b19: A5 -> ~{INT}
- SLOT1 pad b20: A7 -> ~{BUSACK}
- SLOT1 pad b25: unconnected-(SLOT4-Pin_b25-Padb25) -> -12V
- SLOT1 pad b4: unconnected-(SLOT4-Pin_b4-Padb4) -> A5
- SLOT1 pad b5: unconnected-(SLOT4-Pin_b5-Padb5) -> A7
- SLOT1 pad b6: ~{RESET} -> ~{IORQ}
- SLOT1 pad b7: ~{SLOT4} -> ~{IRQ4}
- SLOT1 pad b8: ~{IORQ} -> ~{IRQ6}
- SLOT1 pad b9: ~{IRQ4} -> CLOCK
- SLOT5 pad a5: unconnected-(SLOT5-Pin_a5-Pada5) -> A6
- SLOT5 pad a6: ~{RD} -> ~{WR}
- SLOT5 pad a7: ~{WR} -> ~{IRQ3}
- SLOT5 pad a8: ~{WAIT} -> ~{IRQ5}
- SLOT5 pad a9: CLOCK -> ~{IRQ7}
- SLOT5 pad b1: GND -> +12V
- SLOT5 pad b15: +5V -> GND
- SLOT5 pad b4: unconnected-(SLOT5-Pin_b4-Padb4) -> A5
- SLOT5 pad b5: unconnected-(SLOT5-Pin_b5-Padb5) -> A7
- SLOT5 pad b6: ~{RESET} -> ~{IORQ}
- SLOT5 pad b7: ~{SLOT5} -> ~{IRQ4}
- SLOT5 pad b8: ~{IORQ} -> ~{IRQ6}
- SLOT5 pad b9: ~{IRQ5} -> CLOCK
- U10 pad 1: ~{SLOT1} -> ~{IORQ}
- U10 pad 10: (no net) -> GND
- U10 pad 11: (no net) -> A4
- U10 pad 12: (no net) -> GND
- U10 pad 13: (no net) -> A5
- U10 pad 14: +5V -> GND
- U10 pad 2: ~{RD} -> GND
- U10 pad 3: Net-(U13-~{OE}) -> GND
- U10 pad 4: ~{SLOT1} -> GND
- U10 pad 5: ~{RD} -> GND
- U10 pad 6: Net-(U10-Pad6) -> GND
- U10 pad 8: (no net) -> A3
- U10 pad 9: (no net) -> GND
- U11 pad 1: Net-(J1-Pad5) -> /I/O Controller/~{INTERNAL_IO}
- U11 pad 10: Net-(U11-Pad10) -> unconnected-(U11B-O2-Pad10)
- U11 pad 11: Net-(U11-Pad11) -> unconnected-(U11B-O1-Pad11)
- U11 pad 12: (no net) -> unconnected-(U11B-O0-Pad12)
- U11 pad 13: (no net) -> GND
- U11 pad 14: +5V -> GND
- U11 pad 2: Net-(D1-A) -> A2
- U11 pad 3: Net-(D1-K) -> A1
- U11 pad 4: Net-(U13-RCLK) -> ~{SLOT0}
- U11 pad 5: Net-(C28-Pad1) -> ~{NVRAM}
- U11 pad 6: Net-(U11-Pad6) -> ~{KEYB}
- U11 pad 7: GND -> ~{SERIAL}
- U11 pad 8: Net-(U13-SRCLK) -> GND
- U11 pad 9: Net-(J1-Pad5) -> unconnected-(U11B-O3-Pad9)
- U12 pad 1: Net-(U12-Pad1) -> Net-(U23-P24)
- U12 pad 10: Net-(U11-Pad6) -> Net-(U12-Pad10)
- U12 pad 11: Net-(U11-Pad11) -> (no net)
- U12 pad 12: Net-(U10-Pad6) -> (no net)
- U12 pad 13: ~{RESET} -> (no net)
- U12 pad 2: ~{IRQ1} -> Net-(U23-P25)
- U12 pad 4: Net-(U12-Pad3) -> ~{WR}
- U12 pad 5: Net-(U11-Pad10) -> ~{SLOT0}
- U12 pad 6: ~{IRQ1} -> Net-(U12-Pad6)
- U12 pad 8: Net-(U12-Pad1) -> Net-(U12-Pad8)
- U12 pad 9: Net-(U13-RCLK) -> Net-(U12-Pad6)
- U15 pad 9: ~{SLOT2} -> ~{SERIAL}
- U22 pad 13: /Realtime Clock/~{NVRAM_CS} -> ~{NVRAM}
- U22 pad 19: ~{IRQ3} -> ~{IRQ0}
- U5 pad 20: Net-(JP1-C) -> ~{RAMLO}
- U6 pad 1: ~{WR} -> (no net)
- U6 pad 2: ~{SLOT0} -> (no net)
- U6 pad 3: Net-(U6-Pad3) -> (no net)
- U6 pad 4: Net-(U6-Pad3) -> (no net)
- U6 pad 5: Net-(U6-Pad5) -> (no net)
- U6 pad 6: Net-(U6-Pad6) -> (no net)
- U7 pad 5: Net-(U6-Pad6) -> Net-(U12-Pad8)
- U9 pad 10: (no net) -> AS
- U9 pad 11: (no net) -> A0
- U9 pad 2: /Memory/~{A15} -> Net-(JP1-A)
- U9 pad 4: Net-(U6-Pad5) -> Net-(U12-Pad10)
Routing:
- net -12V: track 0.00 -> 586.9 mm, vias 0 -> 6
- net +5V: track 1188.4 -> 687.4 mm, vias 63 -> 33
- net ~{RD}: track 347.7 -> 0.00 mm, vias 10 -> 0
- net +12V: track 0.00 -> 255.2 mm, vias 0 -> 6
- net ~{IRQ1}: track 226.9 -> 12.5 mm, vias 5 -> 0
- net ~{SLOT0}: track 204.3 -> 0.00 mm, vias 4 -> 0
- net ~{SLOT1}: track 194.6 -> 0.00 mm, vias 7 -> 0
- net ~{INTACK}: track 276.6 -> 85.5 mm, vias 9 -> 0
- net ~{IORQ}: track 285.4 -> 105.7 mm, vias 11 -> 0
- net GND: track 16.4 -> 171.0 mm, vias 2 -> 0
- net ~{IRQ2}: track 148.3 -> 12.5 mm, vias 3 -> 0
- net ~{SLOT2}: track 123.4 -> 0.00 mm, vias 3 -> 0
- net Net-(U12-Pad8): track 0.00 -> 119.9 mm, vias 0 -> 3
- net Net-(U13-RCLK): track 116.5 -> 0.00 mm, vias 11 -> 0
- net D7: track 449.5 -> 334.2 mm, vias 14 -> 9
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Other:
- board text added: "-12V"
- board text added: "Expansion Card"
- board text added: "PCB3D_BR_InterisLogicBoard"
- board text added: "PCB3D_TL_InterisLogicBoard"
- board text added: "github.com/Interis64"
- board text added: "~{RST}"
- board text removed: "-"
- board text removed: "A0"
- board text removed: "A1"
- board text removed: "A10"
- board text removed: "A11"
- board text removed: "A12"
- board text removed: "A13"
- board text removed: "A14"
- board text removed: "A15"
- board text removed: "A2"
- board text removed: "A3"
- board text removed: "A4"
- board text removed: "A5"
- board text removed: "A6"
- board text removed: "A7"
- board text removed: "A8"
- board text removed: "A9"
- board text removed: "CLK"
- board text removed: "D0"
- board text removed: "D1"
- board text removed: "D2"
- board text removed: "D3"
- board text removed: "D4"
- board text removed: "D5"
- board text removed: "D6"
- board text removed: "D7"
- board text removed: "IO Port 0x80 IRQ 0x08"
- board text removed: "IO Port 0xA0 IRQ 0x0A"
- board text removed: "IO Port 0xC0 IRQ 0x0C"
- board text removed: "IO Port 0xE0 IRQ 0x0E"
- board text removed: "Slot4 Card"
- board text removed: "~{BUSACK}"
- board text removed: "~{BUSRQ}"
- board text removed: "~{INTACK}"
- board text removed: "~{INT}"
- board text removed: "~{IORQ}"
- board text removed: "~{IRQ4}"
- board text removed: "~{IRQ5}"
- board text removed: "~{IRQ6}"
- board text removed: "~{IRQ7}"
- board text removed: "~{M1}"
- board text removed: "~{MREQ}"
- board text removed: "~{NMI}"
- board text removed: "~{RD}"
- board text removed: "~{RESET}"
- board text removed: "~{SLOT4}"
- board text removed: "~{SLOT5}"
- board text removed: "~{SLOT6}"
- board text removed: "~{SLOT7}"
- board text removed: "~{WAIT}"
- board text removed: "~{WR}"

Commit message: Work in progress
Parts:
- removed TP1: ~{RES}, TestPoint:TestPoint_Loop_D2.60mm_Drill1.6mm_Beaded
- removed TP2: CLK, TestPoint:TestPoint_Loop_D2.60mm_Drill1.6mm_Beaded
- removed TP4, TP6, TP7: GND, TestPoint:TestPoint_Loop_D2.60mm_Drill1.6mm_Beaded
- JP3: footprint Connector_PinHeader_2.54mm:PinHeader_1x03_P2.54mm_Vertical -> Connector_PinHeader_2.54mm:PinHeader_1x02_P2.54mm_Vertical
- moved JP3 2.52 mm to (252.1, 95.9)
- moved C20 0.68 mm to (97.8, 47.6)
- moved C21 0.68 mm to (104.1, 47.6)
- moved C22 0.68 mm to (97.8, 40.0)
- moved C23 0.68 mm to (104.1, 40.0)
Connections:
- JP3 pad 1: unconnected-(JP3-A-Pad1) -> Net-(JP3-A)
- JP3 pad 2: Net-(JP3-C) -> GND
- U22 pad 21: Net-(JP3-C) -> Net-(JP3-A)
Routing:
- net A0: track 330.9 -> 476.8 mm, vias 4 -> 9
- net +5V: track 687.4 -> 797.5 mm
- net ~{WR}: track 304.0 -> 373.0 mm, vias 7 -> 8
- net /VT82C42 Input/KBD_CLOCK: track 43.1 -> 91.4 mm, vias 1 -> 3
- net Net-(U23-P26): track 0.00 -> 43.2 mm, vias 0 -> 2
- net ~{RESET}: track 407.7 -> 448.4 mm, vias 13 -> 16
- net /VT82C42 Input/MOUSE_CLOCK: track 30.4 -> 69.8 mm, vias 1 -> 3
- net Net-(JP3-A): track 0.00 -> 29.8 mm, vias 0 -> 1
- net Net-(U23-P23): track 0.00 -> 10.2 mm, vias 0 -> 2
- net Net-(U12-Pad6): track 0.00 -> 7.62 mm
- net ~{WAIT}: track 173.1 -> 171.8 mm
- net ~{M1}: track 199.1 -> 198.5 mm
- net D7: track 334.2 -> 333.5 mm
- net CLOCK: track 238.9 -> 239.6 mm
- net A15: track 282.5 -> 281.9 mm
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Other:
- board text added: "A0"
- board text added: "A1"
- board text added: "A10"
- board text added: "A11"
- board text added: "A12"
- board text added: "A13"
- board text added: "A14"
- board text added: "A15"
- board text added: "A2"
- board text added: "A3"
- board text added: "A4"
- board text added: "A5"
- board text added: "A6"
- board text added: "A7"
- board text added: "A8"
- board text added: "A9"
- board text added: "CLK"
- board text added: "D0"
- board text added: "D1"
- board text added: "D2"
- board text added: "D3"
- board text added: "D4"
- board text added: "D5"
- board text added: "D6"
- board text added: "D7"
- board text added: "In"
- board text added: "Out"
- board text added: "~{BUSACK}"
- board text added: "~{BUSRQ}"
- board text added: "~{INTACK}"
- board text added: "~{INT}"
- board text added: "~{IORQ}"
- board text added: "~{IRQ3}"
- board text added: "~{IRQ4}"
- board text added: "~{IRQ5}"
- board text added: "~{IRQ6}"
- board text added: "~{IRQ7}"
- board text added: "~{M1}"
- board text added: "~{MREQ}"
- board text added: "~{NMI}"
- board text added: "~{RD}"
- board text added: "~{RES}"
- board text added: "~{RFSH}"
- board text added: "~{WAIT}"
- board text added: "~{WR}"
- board text added: "—"
