File: Interis 64.kicad_pcb (KiCad board)
At the start: 2 copper layers, 228.6 x 127 mm, 71 parts, among them J2 ExtReset, J3 Conn_01x04, J4 DB9_Male, J5 Conn_01x06, U1 DS1233, U10 74HCT688, U11 74HCT139, U12 74HCT32, U15 MC6850, U16 MAX232, U18 74HCT148, U19 74HCT92, U2 Z80B CPU, U20 74HCT373, U22 DS12885+, U23 VT82C42, U24 74HCT06, U3 28C256, U4 74HCT32, U5 62256, U6 74HCT32, U7 74HCT00, U8 62256, U9 74HCT04, Y1 7.3728MHz, Y2 32.768kHz

Commit message: Finished routing Rev.C
Routing:
- net ~{NVRAM}: track 0.00 -> 283.0 mm, vias 0 -> 7
- net ~{IRQ1}: track 12.5 -> 265.2 mm, vias 0 -> 7
- net ~{IRQ2}: track 12.5 -> 261.9 mm, vias 0 -> 7
- net ~{IORQ}: track 105.7 -> 344.1 mm, vias 0 -> 5
- net AS: track 0.00 -> 194.3 mm, vias 0 -> 4
- net +5V: track 797.5 -> 978.4 mm, vias 33 -> 39
- net ~{RD}: track 0.00 -> 161.1 mm, vias 0 -> 3
- net CLOCK: track 239.6 -> 383.5 mm, vias 2 -> 8
- net ~{INTACK}: track 85.5 -> 221.7 mm, vias 0 -> 4
- net ~{MEMWR}: track 23.9 -> 156.5 mm, vias 0 -> 4
- net D7: track 333.5 -> 459.1 mm, vias 9 -> 15
- net ~{MREQ}: track 105.7 -> 202.9 mm, vias 0 -> 5
- net ~{INT}: track 145.6 -> 234.0 mm, vias 3 -> 5
- net /VT82C42 Input/KBD_DATA: track 0.00 -> 76.2 mm, vias 0 -> 3
- net ~{KEYB}: track 0.00 -> 75.5 mm, vias 0 -> 2
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
Commit message: Layout Tweaks
Parts:
- J2: footprint Connector_JST:JST_XH_B4B-XH-A_1x04_P2.50mm_Vertical -> Connector_PinHeader_2.54mm:PinHeader_1x03_P2.54mm_Vertical
- moved J2 0.87 mm to (38.1, 111.8), turned to 0 degrees
- moved C18 0.63 mm to (189.9, 123.2)
- moved C19 0.63 mm to (192.4, 111.8)
- moved C4 0.63 mm to (165.7, 120.7)
Connections:
- J2 pad 3: GND -> ~{RESET}
Routing:
- net ~{RESET}: track 452.0 -> 447.2 mm, vias 17 -> 16
- net +5V: track 978.4 -> 980.7 mm
- net Net-(BT1-+): track 47.8 -> 49.6 mm, vias 1 -> 3
- net ~{NVRAM}: track 283.0 -> 281.2 mm
- net Net-(LS1--): track 52.9 -> 52.0 mm
- net D0: track 477.2 -> 476.3 mm
- net AS: track 194.3 -> 193.4 mm
- net A3: track 303.3 -> 304.0 mm
- net 64K_MODE: track 40.0 -> 40.6 mm
- net Net-(U12-Pad10): track 111.3 -> 110.8 mm
Other:
- board text removed: "RESET"
