File: Interis 64.kicad_pcb (KiCad board)
At the start: 2 copper layers, 228.6 x 127 mm, 71 parts, among them J2 ExtReset, J3 Conn_01x04, J4 DB9_Male, J5 Conn_01x06, U1 DS1233, U10 74HCT688, U11 74HCT139, U12 74HCT32, U15 MC6850, U16 MAX232, U18 74HCT148, U19 74HCT92, U2 Z80B CPU, U20 74HCT373, U22 DS12885+, U23 VT82C42, U24 74HCT06, U3 28C256, U4 74HCT32, U5 62256, U6 74HCT32, U7 74HCT00, U8 62256, U9 74HCT04, Y1 7.3728MHz, Y2 32.768kHz

Commit message: Add CC lines
Parts:
- added R3: 10k, Resistor_THT:R_Axial_DIN0207_L6.3mm_D2.5mm_P10.16mm_Horizontal, F.Cu at (137.8, 38.7)
- J2: footprint Connector_PinHeader_2.54mm:PinHeader_1x03_P2.54mm_Vertical -> Connector_PinHeader_2.54mm:PinHeader_1x02_P2.54mm_Vertical
- moved REF** 181.8 mm to (34.9, 137.2)
- moved JP3 4.44 mm to (252.1, 100.3)
Connections:
- J2 pad 1: +5V -> GND
- J2 pad 2: GND -> ~{RESET}
- SLOT1 pad a16: unconnected-(SLOT1-Pin_a16-Pada16) -> Net-(SLOT1-Pin_a16)
- SLOT1 pad b16: unconnected-(SLOT1-Pin_b16-Padb16) -> Net-(SLOT1-Pin_b16)
- SLOT2 pad a16: unconnected-(SLOT2-Pin_a16-Pada16) -> Net-(SLOT1-Pin_b16)
- SLOT2 pad b16: unconnected-(SLOT2-Pin_b16-Padb16) -> Net-(SLOT2-Pin_b16)
- SLOT3 pad a16: unconnected-(SLOT3-Pin_a16-Pada16) -> Net-(SLOT2-Pin_b16)
- SLOT3 pad b16: unconnected-(SLOT3-Pin_b16-Padb16) -> Net-(SLOT3-Pin_b16)
- SLOT4 pad a16: unconnected-(SLOT4-Pin_a16-Pada16) -> Net-(SLOT3-Pin_b16)
- SLOT4 pad b16: unconnected-(SLOT4-Pin_b16-Padb16) -> /Slots/CC_OUT4
- SLOT5 pad a16: unconnected-(SLOT5-Pin_a16-Pada16) -> /Slots/CC_OUT4
Routing:
- net Net-(SLOT1-Pin_a16): track 0.00 -> 37.2 mm, vias 0 -> 1
- net Net-(SLOT3-Pin_b16): track 0.00 -> 15.2 mm
- net Net-(SLOT2-Pin_b16): track 0.00 -> 15.2 mm
- net Net-(SLOT1-Pin_b16): track 0.00 -> 15.2 mm
- net /Slots/CC_OUT4: track 0.00 -> 15.2 mm
- net +5V: track 980.7 -> 975.6 mm, vias 39 -> 38
- net Net-(JP3-A): track 29.8 -> 25.4 mm
- net ~{RESET}: track 447.2 -> 444.6 mm
Other:
- board text added: "CC IN"
- board text added: "CC OUT"
- board text added: "Clear NVRAM"
- board text removed: "Assembled:"
- board text removed: "—"
