File: Power.kicad_sch (KiCad schematic)
At the start: 41 parts, among them J7 POWER, U10 74HC32, U11 74HC14, U12 74HC00, U4 74HC32, U6 74HC32, U7 74HC00, U9 74HC04

Commit message: Schematic cleanup
Parts:
- removed H1, H2, H3, H4, H5, H6: MountingHole_Pad, MountingHole:MountingHole_3.2mm_M3_Pad_Via, symbol Mechanical:MountingHole_Pad
- added U21: 74HC02, Package_DIP:DIP-14_W7.62mm_LongPads, symbol 74xx:74HC02
Connections:
- net +5V: now also U21.14 (VCC)
- net GND: now also U21.7 (GND)
Other:
- note removed: "Mounting Holes"
- moved on the sheet: C10, C11, C12, C13, C14, C15, C16, C17, C18, C19, C2, C3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

Commit message: Misc Updates/Cleanup
Parts:
- TP3, TP4, TP5, TP6, TP7, TP8: footprint TestPoint:TestPoint_THTPad_2.5x2.5mm_Drill1.2mm -> TestPoint:TestPoint_Loop_D2.60mm_Drill1.6mm_Beaded
- U10, U4, U6: value 74HC32 -> 74HCT32
- U11: value 74HC14 -> 74HCT14
- U12, U7: value 74HC00 -> 74HCT00
- U21: value 74HC02 -> 74HCT02
- U9: value 74HC04 -> 74HCT04
Changed lines of the file:
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@@
       (effects (font (size 1.27 1.27)) (justify left))
     )
-    (property "Value" "74HC32" (at 114.3 95.25 0)
+    (property "Value" "74HCT32" (at 114.3 95.25 0)
       (effects (font (size 1.27 1.27)) (justify left))
     )
@@
       (effects (font (size 1.27 1.27)) (justify left))
     )
-    (property "Value" "74HC14" (at 132.08 95.25 0)
+    (property "Value" "74HCT14" (at 132.08 95.25 0)
       (effects (font (size 1.27 1.27)) (justify left))
     )
@@
       (effects (font (size 1.27 1.27)))
     )
-    (property "Footprint" "TestPoint:TestPoint_THTPad_2.5x2.5mm_Drill1.2mm" (at 45.72 167.005 0)
+    (property "Footprint" "TestPoint:TestPoint_Loop_D2.60mm_Drill1.6mm_Beaded" (at 45.72 167.005 0)
       (effects (font (size 1.27 1.27)) hide)
     )
@@
       (effects (font (size 1.27 1.27)))
     )
-    (property "Footprint" "TestPoint:TestPoint_THTPad_2.5x2.5mm_Drill1.2mm" (at 45.72 141.605 0)
+    (property "Footprint" "TestPoint:TestPoint_Loop_D2.60mm_Drill1.6mm_Beaded" (at 45.72 141.605 0)
       (effects (font (size 1.27 1.27)) hide)
     )
@@
       (effects (font (size 1.27 1.27)))
     )
-    (property "Footprint" "TestPoint:TestPoint_THTPad_2.5x2.5mm_Drill1.2mm" (at 45.72 154.305 0)
+    (property "Footprint" "TestPoint:TestPoint_Loop_D2.60mm_Drill1.6mm_Beaded" (at 45.72 154.305 0)
       (effects (font (size 1.27 1.27)) hide)
     )
@@
       (effects (font (size 1.27 1.27)))
     )
-    (property "Footprint" "TestPoint:TestPoint_THTPad_2.5x2.5mm_Drill1.2mm" (at 45.72 160.655 0)
+    (property "Footprint" "TestPoint:TestPoint_Loop_D2.60mm_Drill1.6mm_Beaded" (at 45.72 160.655 0)
       (effects (font (size 1.27 1.27)) hide)
     )
@@
       (effects (font (size 1.27 1.27)))
     )
-    (property "Value" "74HC04" (at 194.31 95.25 0)
+    (property "Value" "74HCT04" (at 194.31 95.25 0)
       (effects (font (size 1.27 1.27)))
     )
@@
       (effects (font (size 1.27 1.27)))
     )
-    (property "Value" "74HC00" (at 175.26 95.25 0)
+    (property "Value" "74HCT00" (at 175.26 95.25 0)
       (effects (font (size 1.27 1.27)))
     )
@@
       (effects (font (size 1.27 1.27)))
     )
-    (property "Value" "74HC32" (at 156.21 95.25 0)
+    (property "Value" "74HCT32" (at 156.21 95.25 0)
       (effects (font (size 1.27 1.27)))
     )
@@
       (effects (font (size 1.27 1.27)))
     )
-    (property "Footprint" "TestPoint:TestPoint_THTPad_2.5x2.5mm_Drill1.2mm" (at 45.72 173.355 0)
+    (property "Footprint" "TestPoint:TestPoint_Loop_D2.60mm_Drill1.6mm_Beaded" (at 45.72 173.355 0)
       (effects (font (size 1.27 1.27)) hide)
     )
@@
       (effects (font (size 1.27 1.27)))
     )
-    (property "Footprint" "TestPoint:TestPoint_THTPad_2.5x2.5mm_Drill1.2mm" (at 45.72 147.955 0)
+    (property "Footprint" "TestPoint:TestPoint_Loop_D2.60mm_Drill1.6mm_Beaded" (at 45.72 147.955 0)
       (effects (font (size 1.27 1.27)) hide)
     )
@@
       (effects (font (size 1.27 1.27)))
     )
-    (property "Value" "74HC00" (at 83.82 95.25 0)
+    (property "Value" "74HCT00" (at 83.82 95.25 0)
       (effects (font (size 1.27 1.27)))
     )
@@
       (effects (font (size 1.27 1.27)))
     )
-    (property "Value" "74HC02" (at 68.58 95.25 0)
+    (property "Value" "74HCT02" (at 68.58 95.25 0)
       (effects (font (size 1.27 1.27)))
     )
@@
       (effects (font (size 1.27 1.27)))
     )
-    (property "Value" "74HC32" (at 100.33 95.25 0)
-      (effects (font (size 1.27 1.27)))
-    )
+    (property "Value" "74HCT32" (at 100.33 95.25 0)
+      (effects (font (size 1.27 1.27)))
+    )

Commit message: Work-in-progress
Parts:
- removed C12, C13, C31: 0.1µF, Capacitor_THT:C_Disc_D5.0mm_W2.5mm_P2.50mm, symbol Device:C
- removed J7: POWER, Connector_TE-Connectivity:TE_MATE-N-LOK_350211-1_1x04_P5.08mm_Vertical, symbol Connector_Generic:Conn_01x04
- removed TP3, TP5, TP8: GND, TestPoint:TestPoint_Loop_D2.60mm_Drill1.6mm_Beaded, symbol Connector:TestPoint
- removed U10: 74HCT32, Package_DIP:DIP-14_W7.62mm_LongPads, symbol 74xx:74LS32
- removed U11: 74HCT14, Package_DIP:DIP-14_W7.62mm_LongPads, symbol 74xx:74LS14
- removed U21: 74HCT02, Package_DIP:DIP-14_W7.62mm_LongPads, symbol 74xx:74HC02
- added J3: Conn_01x04, Interis-Footprints:TE_EconomyPower_1744037-x_1x04_P5.08mm_Vertical, symbol Connector_Generic:Conn_01x04
- U12: value 74HCT00 -> 74HCT32; footprint Package_DIP:DIP-14_W7.62mm_LongPads -> Package_DIP:DIP-14_W7.62mm
- U4, U6, U7, U9: footprint Package_DIP:DIP-14_W7.62mm_LongPads -> Package_DIP:DIP-14_W7.62mm
Connections:
- net +12V: now also J3.3 (Pin_3)
- net +5V: now also J3.1 (Pin_1)
- net GND: now also J3.2 (Pin_2)
- new net -12V: J3.4 (Pin_4)

Commit message: Work in progress
Parts:
- removed TP4, TP6, TP7: GND, TestPoint:TestPoint_Loop_D2.60mm_Drill1.6mm_Beaded, symbol Connector:TestPoint
Other:
- note removed: "Test Point Grounds"
Changed lines of the file:
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@@
   (junction (at 93.98 31.75) (diameter 0) (color 0 0 0 0)
   )
-  (junction (at 45.72 172.085) (diameter 0) (color 0 0 0 0)
-  )
   (junction (at 73.66 31.75) (diameter 0) (color 0 0 0 0)
   )
@@
   (junction (at 104.14 31.75) (diameter 0) (color 0 0 0 0)
   )
-  (junction (at 45.72 178.435) (diameter 0) (color 0 0 0 0)
-  )
   (junction (at 43.18 31.75) (diameter 0) (color 0 0 0 0)
   )
@@
   (junction (at 190.5 39.37) (diameter 0) (color 0 0 0 0)
   )
-  (junction (at 45.72 159.385) (diameter 0) (color 0 0 0 0)
-  )
   (junction (at 53.34 31.75) (diameter 0) (color 0 0 0 0)
   )
@@
     (stroke (width 0) (type default))
   )
-  (wire (pts (xy 45.72 172.085) (xy 45.72 178.435))
-    (stroke (width 0) (type default))
-  )
   (wire (pts (xy 83.82 107.95) (xy 118.11 107.95))
     (stroke (width 0) (type default))
@@
     (stroke (width 0) (type default))
   )
-  (wire (pts (xy 45.72 178.435) (xy 45.72 179.705))
-    (stroke (width 0) (type default))
-  )
   (wire (pts (xy 168.91 31.75) (xy 158.75 31.75))
     (stroke (width 0) (type default))
   )
-  (wire (pts (xy 45.72 146.685) (xy 45.72 159.385))
-    (stroke (width 0) (type default))
-  )
   (wire (pts (xy 53.34 31.75) (xy 43.18 31.75))
     (stroke (width 0) (type default))
@@
     (stroke (width 0) (type default))
   )
-  (wire (pts (xy 45.72 159.385) (xy 45.72 172.085))
-    (stroke (width 0) (type default))
-  )
   (wire (pts (xy 83.82 39.37) (xy 93.98 39.37))
     (stroke (width 0) (type default))
@@
   )
   (text "Power Connector" (at 101.6 191.135 0)
-    (effects (font (size 2.54 2.54)) (justify left bottom))
-  )
-  (text "Test Point Grounds" (at 29.21 191.77 0)
     (effects (font (size 2.54 2.54)) (justify left bottom))
   )
@@
     )
   )
-  (symbol (lib_id "power:GND") (at 45.72 179.705 0) (unit 1)
-    (in_bom yes) (on_board yes) (dnp no)
-    (property "Reference" "#PWR024" (at 45.72 186.055 0)
-      (effects (font (size 1.27 1.27)) hide)
-    )
-    (property "Value" "GND" (at 45.847 184.0992 0)
-      (effects (font (size 1.27 1.27)))
-    )
-    (property "Footprint" "" (at 45.72 179.705 0)
-      (effects (font (size 1.27 1.27)) hide)
-    )
-    (property "Datasheet" "" (at 45.72 179.705 0)
-      (effects (font (size 1.27 1.27)) hide)
-    )
-    (pin "1")
-    (instances
-      (project "Interis 64"
-        (path "/b7aa0362-7c9e-4a42-b191-ab15a38bf3c5/00000000-0000-0000-0000-000062c2416e"
-          (reference "#PWR024") (unit 1)
-        )
-      )
-    )
-  )
   (symbol (lib_id "power:-12V") (at 129.54 156.845 0) (unit 1)
     (in_bom yes) (on_board yes) (dnp no) (fields_autoplaced)
@@
     )
   )
-  (symbol (lib_id "Connector:TestPoint") (at 45.72 172.085 90) (unit 1)
-    (in_bom yes) (on_board yes) (dnp no) (fields_autoplaced)
-    (property "Reference" "TP6" (at 42.418 167.7502 90)
-      (effects (font (size 1.27 1.27)))
-    )
-    (property "Value" "GND" (at 42.418 170.2871 90)
-      (effects (font (size 1.27 1.27)))
-    )
-    (property "Footprint" "TestPoint:TestPoint_Loop_D2.60mm_Drill1.6mm_Beaded" (at 45.72 167.005 0)
-      (effects (font (size 1.27 1.27)) hide)
-    )
-    (property "Datasheet" "~" (at 45.72 167.005 0)
-      (effects (font (size 1.27 1.27)) hide)
-    )
-    (pin "1")
-    (instances
-      (project "Interis 64"
-        (path "/b7aa0362-7c9e-4a42-b191-ab15a38bf3c5/00000000-0000-0000-0000-000062c2416e"
-          (reference "TP6") (unit 1)
-        )
-      )
-    )
-  )
   (symbol (lib_id "Device:C") (at 168.91 35.56 0) (unit 1)
     (in_bom yes) (on_board yes) (dnp no)
@@
         (path "/b7aa0362-7c9e-4a42-b191-ab15a38bf3c5/00000000-0000-0000-0000-000062c2416e"
           (reference "C19") (unit 1)
-        )
-      )
-    )
-  )
-  (symbol (lib_id "Connector:TestPoint") (at 45.72 159.385 90) (unit 1)
-    (in_bom yes) (on_board yes) (dnp no) (fields_autoplaced)
-    (property "Reference" "TP4" (at 42.418 155.0502 90)
-      (effects (font (size 1.27 1.27)))
-    )
-    (property "Value" "GND" (at 42.418 157.5871 90)
-      (effects (font (size 1.27 1.27)))
-    )
-    (property "Footprint" "TestPoint:TestPoint_Loop_D2.60mm_Drill1.6mm_Beaded" (at 45.72 154.305 0)
-      (effects (font (size 1.27 1.27)) hide)
-    )
-    (property "Datasheet" "~" (at 45.72 154.305 0)
-      (effects (font (size 1.27 1.27)) hide)
-    )
-    (pin "1")
-    (instances
-      (project "Interis 64"
-        (path "/b7aa0362-7c9e-4a42-b191-ab15a38bf3c5/00000000-0000-0000-0000-000062c2416e"
-          (reference "TP4") (unit 1)
         )
       )
@@
         )
       )
-    )
-  )
-  (symbol (lib_id "Connector:TestPoint") (at 45.72 178.435 90) (unit 1)
-    (in_bom yes) (on_board yes) (dnp no) (fields_autoplaced)
-    (property "Reference" "TP7" (at 42.418 174.1002 90)
-      (effects (font (size 1.27 1.27)))
-    )
-    (property "Value" "GND" (at 42.418 176.6371 90)
-      (effects (font (size 1.27 1.27)))
-    )
-    (property "Footprint" "TestPoint:TestPoint_Loop_D2.60mm_Drill1.6mm_Beaded" (at 45.72 173.355 0)
-      (effects (font (size 1.27 1.27)) hide)
-    )
-    (property "Datasheet" "~" (at 45.72 173.355 0)
-      (effects (font (size 1.27 1.27)) hide)
-    )
-    (pin "1")
-    (instances
-      (project "Interis 64"
-        (path "/b7aa0362-7c9e-4a42-b191-ab15a38bf3c5/00000000-0000-0000-0000-000062c2416e"
-          (reference "TP7") (unit 1)
-        )
-      )
