File: VT82C42.kicad_sch (KiCad schematic)
At the start: 4 parts, among them J5 Conn_01x06, U12 74HCT32, U23 VT82C42, U24 74HCT06

Commit message: Work in progress
Other:
- moved on the sheet: U24F
Changed lines of the file:
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@@
     (stroke (width 0) (type default))
   )
-  (wire (pts (xy 69.215 111.76) (xy 83.185 111.76))
+  (wire (pts (xy 65.405 111.76) (xy 83.185 111.76))
     (stroke (width 0) (type default))
   )
@@
     (stroke (width 0) (type default))
   )
-  (wire (pts (xy 59.69 90.17) (xy 83.185 90.17))
+  (wire (pts (xy 65.405 90.17) (xy 83.185 90.17))
     (stroke (width 0) (type default))
   )
@@
     (stroke (width 0) (type default))
   )
+  (wire (pts (xy 39.37 90.17) (xy 50.165 90.17))
+    (stroke (width 0) (type default))
+  )
   (wire (pts (xy 200.025 50.165) (xy 219.71 50.165))
     (stroke (width 0) (type default))
@@
     (stroke (width 0) (type default))
   )
-  (wire (pts (xy 205.105 130.175) (xy 219.71 130.175))
+  (wire (pts (xy 205.105 130.175) (xy 234.315 130.175))
     (stroke (width 0) (type default))
   )
@@
     (stroke (width 0) (type default))
   )
-  (wire (pts (xy 202.565 120.015) (xy 219.71 120.015))
+  (wire (pts (xy 202.565 120.015) (xy 234.315 120.015))
     (stroke (width 0) (type default))
   )
@@
     (effects (font (size 1.27 1.27)) (justify right bottom))
   )
-  (label "KBD_DATA" (at 219.71 130.175 180) (fields_autoplaced)
+  (label "KBD_DATA" (at 234.315 130.175 180) (fields_autoplaced)
     (effects (font (size 1.27 1.27)) (justify right bottom))
   )
@@
     (effects (font (size 1.27 1.27)) (justify right bottom))
   )
-  (label "KBD_CLOCK" (at 219.71 120.015 180) (fields_autoplaced)
+  (label "KBD_CLOCK" (at 234.315 120.015 180) (fields_autoplaced)
     (effects (font (size 1.27 1.27)) (justify right bottom))
   )
@@
     (effects (font (size 1.27 1.27)) (justify right bottom))
   )
-  (global_label "CLOCK" (shape input) (at 69.215 111.76 180) (fields_autoplaced)
+  (global_label "CLOCK" (shape input) (at 65.405 111.76 180) (fields_autoplaced)
     (effects (font (size 1.27 1.27)) (justify right))
-    (property "Intersheetrefs" "${INTERSHEET_REFS}" (at 60.7222 111.6806 0)
+    (property "Intersheetrefs" "${INTERSHEET_REFS}" (at 56.9122 111.6806 0)
       (effects (font (size 1.27 1.27)) (justify right) hide)
     )
   )
-  (global_label "~{WR}" (shape bidirectional) (at 44.45 90.17 180) (fields_autoplaced)
+  (global_label "~{WR}" (shape bidirectional) (at 39.37 90.17 180) (fields_autoplaced)
     (effects (font (size 1.27 1.27)) (justify right))
-    (property "Intersheetrefs" "${INTERSHEET_REFS}" (at 37.8893 90.17 0)
+    (property "Intersheetrefs" "${INTERSHEET_REFS}" (at 32.8093 90.17 0)
       (effects (font (size 1.27 1.27)) (justify right) hide)
     )
@@
     )
   )
-  (symbol (lib_id "74xx:74LS06") (at 52.07 90.17 0) (unit 6)
+  (symbol (lib_id "74xx:74LS06") (at 57.785 90.17 0) (unit 6)
     (in_bom yes) (on_board yes) (dnp no) (fields_autoplaced)
-    (property "Reference" "U24" (at 52.07 83.3501 0)
-      (effects (font (size 1.27 1.27)))
-    )
-    (property "Value" "74HCT06" (at 52.07 85.2711 0)
-      (effects (font (size 1.27 1.27)))
-    )
-    (property "Footprint" "Package_DIP:DIP-14_W7.62mm" (at 52.07 90.17 0)
-      (effects (font (size 1.27 1.27)) hide)
-    )
-    (property "Datasheet" "http://www.ti.com/lit/gpn/sn74LS06" (at 52.07 90.17 0)
-      (effects (font (size 1.27 1.27)) hide)
-    )
+    (property "Reference" "U24" (at 57.785 83.3501 0)
+      (effects (font (size 1.27 1.27)))
+    )
+    (property "Value" "74HCT06" (at 57.785 85.2711 0)
+      (effects (font (size 1.27 1.27)))
+    )
+    (property "Footprint" "Package_DIP:DIP-14_W7.62mm" (at 57.785 90.17 0)
+      (effects (font (size 1.27 1.27)) hide)
+    )
+    (property "Datasheet" "http://www.ti.com/lit/gpn/sn74LS06" (at 57.785 90.17 0)
+      (effects (font (size 1.27 1.27)) hide)
+    )
